File: pcb/HM-LC-SW1-PCB.sch (EAGLE design)
At the start: 15 parts, among them IC1 CC1101, IC2 ITS428L2, T1 MTD3055E

Commit message: Schaltplan
Schaltplan weiter gemacht
Parts:
- added IC3: LP2950Z, linear:LP2950Z
- added R2: 100k, 1WIDER:WIDERSAND
- added SJ3, SJ4: (no value), jumper:SJ
Connections:
- new net N$11: R2.2, U$1.D5
- new net V+: +VCC.1, C1.2, C2.+, IC2.VBB, IC3.I, SJ2.1, SJ3.1, SJ4.1
- net +3V3: now also IC3.O, SJ4.2
- net GND: now also IC3.GND
- net N$6: now also R2.1; no longer U$1.D5
- net VCC: now also SJ3.2; no longer +VCC.1, C1.2, C2.+, IC2.VBB, SJ2.1
Other:
- moved on the sheet: +VCC, C1, C2, GND, IC2, OUT+, OUTGND, SJ1, SJ2, T1

Commit message: Layout V1
Layout fertig
Parts:
- removed +VCC, GND: (no value), 3PASSIVE:LÖTPAD
- removed OUT+, OUTGND: PIN, 3PASSIVE:PIN
- removed SJ1, SJ2: (no value), jumper:SJ
- removed T1: MTD3055E, 8TRANSIS:MTD3055E
- added ANT: (no value), 3PASSIVE:LÖTPAD
- added LED2: (no value), LED:LED3MM
- added R4: 330, 1WIDER:WIDERSAND
- added X1: (no value), con-phoenix-381_l:MCV4
Connections:
- removed net N$10: OUTGND.1, SJ1.2, T1.DRA
- new net N$14: LED2.ANO, R4.1
- net GND: now also IC1.GNDA1, IC1.GNDA2, LED2.KAT, X1.2.SK, X1.4.SK; no longer GND.1, SJ1.1, T1.SO
- net N$11: now also R4.2
- net N$13: now also ANT.1
- net N$6: no longer T1.GAA
- net OUT: now also X1.3.SK; no longer OUT+.1, SJ2.2
- net V+: now also X1.1.SK; no longer +VCC.1, SJ2.1
Other:
- moved on the sheet: CONFIG, LED1, R1
